File: Hardware/SparkFun_GNSS_UM980.kicad_pcb (KiCad board)
At the start: 4 copper layers, 50.8 x 50.8 mm, 142 parts, among them J1 USB_C_Receptacle, J4 Conn_01x02, J5 SMA_EdgeMount, J6 JST_Locking_4, J7 Conn_01x06, J8 Conn_01x09, U1 TVS_DIODE_ARRAY, U2 AP2112K-3.3, U5 UM980, U8 CH340C

Commit message: Post design review.
Parts:
- removed the G*** at (127.0, 120.7)
- removed kibuzzard-64C2E9F4: G***, kibuzzard-64C2E9F4
- removed kibuzzard-64C2E9F9: G***, kibuzzard-64C2E9F9
- removed kibuzzard-64C2E9FD: G***, kibuzzard-64C2E9FD
- removed kibuzzard-64E77485: G***, kibuzzard-64E77485
- removed kibuzzard-64E7748C: G***, kibuzzard-64E7748C
- added G***: LOGO, SparkFun-Aesthetic:SparkFun_Logo_20mm, B.Cu at (127.0, 120.7)
- added JP8: BT-VCC, SparkFun-Jumper:SMT-JUMPER_2_NC_TRACE_SILK, B.Cu at (132.1, 142.2)
- added R8: 1k, SparkFun-Resistor:R_0603_1608Metric, F.Cu at (114.3, 147.3)
- added Ref**: Val**, SparkFun-Aesthetic:OSHW_Logo_5mm, B.Cu at (148.6, 142.2)
- added kibuzzard-65087150: G***, kibuzzard-65087150, F.Cu at (133.3, 148.7)
- added kibuzzard-65087158: G***, kibuzzard-65087158, B.Cu at (133.3, 148.7)
- added kibuzzard-650880D6: G***, kibuzzard-650880D6, B.Cu at (127.0, 125.7)
- added kibuzzard-650880DF: G***, kibuzzard-650880DF, B.Cu at (127.0, 129.5)
- added kibuzzard-650880E6: G***, kibuzzard-650880E6, B.Cu at (127.0, 133.3)
- added kibuzzard-650885D8: G***, kibuzzard-650885D8, B.Cu at (136.4, 142.2)
- BT1: value 6.8mm_Coin_Cell -> ML414H
- U7: footprint SparkFun-Aesthetic:Ordering_Instructions -> SparkFun-Aesthetic:ORDERING_INSTRUCTIONS
- moved D6 1.27 mm to (144.8, 132.0)
- moved L1 0.90 mm to (143.4, 130.9), turned to -90 degrees
- moved U7 0.28 mm to (165.2, 101.8)
Connections:
- J6 pad 2: RXD2 -> Net-(J6-Pin_2)
- J7 pad 4: +3.3V -> Net-(J7-Pin_4)
Routing:
- net RXD2: track 64.9 -> 54.1 mm
- net Net-(J6-Pin_2): track 0.00 -> 10.2 mm
- net Net-(J7-Pin_4): track 0.00 -> 9.20 mm
- net Net-(D6-A2): track 7.97 -> 6.61 mm
- net +3.3V: track 86.0 -> 85.2 mm
- added copper zone on In2.Cu, net GND

Commit message: Update to v8. Update models.
Parts:
- BT1: value ML414H -> 6.8mm_ML414H
- D1: footprint SparkFun-LED:LED_0603_1608Metric -> SparkFun-LED:LED_0603_1608Metric_Red
- D2: footprint SparkFun-LED:LED_0603_1608Metric -> SparkFun-LED:LED_0603_1608Metric_White
- D3: footprint SparkFun-LED:LED_0603_1608Metric -> SparkFun-LED:LED_0603_1608Metric_Blue
- D4: footprint SparkFun-LED:LED_0603_1608Metric -> SparkFun-LED:LED_0603_1608Metric_Yellow
- D6: value PESD0402 -> PESD0402
- FID1, FID2, FID3, FID4: value Fiducial_0.5 -> Fiducial_0.5mm
- J1: footprint SparkFun-Connector:USB-C-16P -> SparkFun-Connector:USB-C_16
- J4: footprint SparkFun-Connector:1X02 -> SparkFun-Connector:1x02
- J5: value SMA_EdgeMount -> SMA_Edge; footprint SparkFun-Connector:SMA-EDGE -> SparkFun-Connector:SMA_Edge
- J6: footprint SparkFun-Connector:JST-4-SMD-1.25MM-LOCKING -> SparkFun-Connector:JST_SMD_1.25mm-4_Locking
- J7: footprint SparkFun-Connector:1X06 -> SparkFun-Connector:1x06
- J8: footprint SparkFun-Connector:1X09 -> SparkFun-Connector:1x09
- JP1, JP6: footprint SparkFun-Jumper:SMT-JUMPER_3_1-NC_TRACE_SILK -> SparkFun-Jumper:Jumper_3_NC-1_Trace
- JP2, JP3, JP4, JP5, JP7: footprint SparkFun-Jumper:SMT-JUMPER_2_NC_TRACE_SILK -> SparkFun-Jumper:Jumper_2_NC_Trace
- JP8: value BT-VCC -> ~; footprint SparkFun-Jumper:SMT-JUMPER_2_NC_TRACE_SILK -> SparkFun-Jumper:Jumper_2_NC_Trace
- L2: value 30Ω -> 30Ohm
- ST1, ST2, ST3, ST4: value Stand_off -> Standoff; footprint SparkFun-Hardware:STAND-OFF -> SparkFun-Hardware:Standoff
- TP1, TP2: value TestPoint -> PTH; footprint SparkFun-Connector:1X01 -> SparkFun-Connector:1x01
- U1: value TVS_DIODE_ARRAY -> DT1042-04SO
- U7: footprint SparkFun-Aesthetic:ORDERING_INSTRUCTIONS -> SparkFun-Aesthetic:Ordering_Instructions
- U8: footprint SparkFun-Semiconductor-Standard:SO16 -> SparkFun-Semiconductor-Standard:SO-16
- turned R32 to -90 degrees
- turned R33 to -90 degrees
Connections:
- net +3.3V renamed 3.3V
- net +3.3V_A renamed 3.3V_A
- J5 pad 1: GND -> Net-(D6-A2)
- R32 pad 1: Net-(U5-BIF_28) -> Net-(R14-Pad2)
- R32 pad 2: Net-(R14-Pad2) -> Net-(U5-BIF_28)
- R33 pad 1: Net-(U5-BIF_29) -> Net-(R13-Pad2)
- R33 pad 2: Net-(R13-Pad2) -> Net-(U5-BIF_29)
