File: Hardware/SparkFun_GNSS_UM980.kicad_sch (KiCad schematic)
At the start: 66 parts, among them J1 USB_C_Receptacle, U1 TVS_DIODE_ARRAY, U2 AP2112K-3.3, U5 UM980, U8 CH340C

Commit message: Post design review.
Parts:
- BT1: value 6.8mm_Coin_Cell -> ML414H; symbol SparkFun-Battery:BATTERY_6.8mm_ML414H_IV01E -> SparkFun-Battery:Battery_6.8mm_ML414H_IV01E
- D1: PROD_ID DIO-00819 -> DIO-17976
- U7: footprint SparkFun-Aesthetic:Ordering_Instructions -> SparkFun-Aesthetic:ORDERING_INSTRUCTIONS
Connections:
- net at J1.A8 (NC): now also J1.B8 (NC)
- net at J1.NC1 (NC): now also J1.NC2 (NC), J1.NC3 (NC)

Commit message: Update to v8. Update models.
Parts:
- BT1: value ML414H -> 6.8mm_ML414H
- C1, C16, C2: Tolerance +80%/-20% -> 20%; Voltage 25 -> 25V
- D1: footprint SparkFun-LED:LED_0603_1608Metric -> SparkFun-LED:LED_0603_1608Metric_Red
- D2: footprint SparkFun-LED:LED_0603_1608Metric -> SparkFun-LED:LED_0603_1608Metric_White
- D3: footprint SparkFun-LED:LED_0603_1608Metric -> SparkFun-LED:LED_0603_1608Metric_Blue
- D4: footprint SparkFun-LED:LED_0603_1608Metric -> SparkFun-LED:LED_0603_1608Metric_Yellow
- D5: IMax (none) -> 0.5A; VDrop (none) -> 0.42V; VMax (none) -> 40V
- FID1, FID2, FID3, FID4: value Fiducial_0.5 -> Fiducial_0.5mm; symbol SparkFun-Aesthetic:Fiducial_0.5 -> SparkFun-Aesthetic:Fiducial_0.5mm
- J1: footprint SparkFun-Connector:USB-C-16P -> SparkFun-Connector:USB-C_16
- JP2, JP3, JP4, JP5, JP7: footprint SparkFun-Jumper:SMT-JUMPER_2_NC_TRACE_SILK -> SparkFun-Jumper:Jumper_2_NC_Trace
- L2: value 30Ω -> 30Ohm; symbol SparkFun-Coil:30Ohm_100MHz_0603 -> SparkFun-Coil:30Ohm_0603_1.8A
- ST1, ST2, ST3, ST4: value Stand_off -> Standoff; footprint SparkFun-Hardware:STAND-OFF -> SparkFun-Hardware:Standoff; symbol SparkFun-Hardware:Stand_off -> SparkFun-Hardware:Standoff
- TP1, TP2: value TestPoint -> PTH; footprint SparkFun-Connector:1X01 -> SparkFun-Connector:1x01
- U1: value TVS_DIODE_ARRAY -> DT1042-04SO
- U2: Imax (none) -> 600mA; Iq (none) -> 55µA; VMax (none) -> 6V
- U7: footprint SparkFun-Aesthetic:ORDERING_INSTRUCTIONS -> SparkFun-Aesthetic:Ordering_Instructions
- U8: footprint SparkFun-Semiconductor-Standard:SO16 -> SparkFun-Semiconductor-Standard:SO-16
Connections:
- net at R13.2, TP1.1: now also R33.1; no longer R33.2
- net at R32.1: now also R14.2, TP2.1; no longer U5.28 (BIF_28)
- net at U5.29 (BIF_29): now also R33.2; no longer R33.1
- net +3.3V renamed 3.3V
- net +3.3V_A renamed 3.3V_A
- new net: R32.2, U5.28 (BIF_28)
Other:
- moved on the sheet: F1, R1, R12, R13, R14, R15, R16, R17, R18, R19, R2, R20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
